File: Kicad Project/RS232-USB_SerialConverter.sch (KiCad schematic (older format))
At the start: 9 parts

Commit message: add pcb
Parts:
- C1, C2, C3, C4, C5: renamed from C?; footprint (none) -> Capacitors_SMD:C_0603_HandSoldering
- J1: renamed from J?; footprint (none) -> MyLib:D-SUB Position 9 rightangle
- J2: renamed from J?; footprint (none) -> Pin_Headers:Pin_Header_Straight_1x06_Pitch2.54mm
- JP1: renamed from JP?; footprint (none) -> Pin_Headers:Pin_Header_Straight_1x02_Pitch2.54mm
- U1: renamed from U?; footprint (none) -> Housings_SOIC:SOIC-16W_5.3x10.2mm_Pitch1.27mm
Changed lines of the file:
@@
 LIBS:valves
 LIBS:Mylib
+LIBS:RS232-USB_SerialConverter-cache
 EELAYER 25 0
 EELAYER END
@@
 $EndDescr
 $Comp
-L Conn_01x09_Male J?
+L Conn_01x09_Male J1
 U 1 1 5B22F1AF
 P 3850 3100
-F 0 "J?" H 3850 3600 50  0000 C CNN
+F 0 "J1" H 3850 3600 50  0000 C CNN
 F 1 "TIA/EIA-232-Male" H 3850 2600 50  0000 C CNN
-F 2 "" H 3850 3100 50  0001 C CNN
+F 2 "MyLib:D-SUB Position 9 rightangle" H 3850 3100 50  0001 C CNN
 F 3 "" H 3850 3100 50  0001 C CNN
 	1    3850 3100
@@
 Pin1 Data Carrier Detect(DCD)\nPin2 Recieved Data(RD)\nPin3 Transmit Data(TD)\nPin4 Data Terminal Ready(DTR)\nPin5 Signal Ground(SG)\nPin6 Data Set Ready(DSR)\nPin7 Request To Send(RTS)\nPin8 Clear To Send(CTS)\nPin9 Ring Indicator(RI)
 $Comp
-L GND #PWR?
+L GND #PWR01
 U 1 1 5B22F353
 P 4550 3950
-F 0 "#PWR?" H 4550 3700 50  0001 C CNN
+F 0 "#PWR01" H 4550 3700 50  0001 C CNN
 F 1 "GND" H 4550 3800 50  0000 C CNN
 F 2 "" H 4550 3950 50  0001 C CNN
@@
 NoConn ~ 4050 3500
 $Comp
-L C C?
+L C C2
 U 1 1 5B22F4AD
 P 7100 2900
-F 0 "C?" H 7125 3000 50  0000 L CNN
+F 0 "C2" H 7125 3000 50  0000 L CNN
 F 1 "0.1uF" H 7125 2800 50  0000 L CNN
-F 2 "" H 7138 2750 50  0001 C CNN
+F 2 "Capacitors_SMD:C_0603_HandSoldering" H 7138 2750 50  0001 C CNN
 F 3 "" H 7100 2900 50  0001 C CNN
 	1    7100 2900
@@
 $EndComp
 $Comp
-L C C?
+L C C1
 U 1 1 5B22F4D4
 P 5100 2900
-F 0 "C?" H 5125 3000 50  0000 L CNN
+F 0 "C1" H 5125 3000 50  0000 L CNN
 F 1 "0.1uF" H 5125 2800 50  0000 L CNN
-F 2 "" H 5138 2750 50  0001 C CNN
+F 2 "Capacitors_SMD:C_0603_HandSoldering" H 5138 2750 50  0001 C CNN
 F 3 "" H 5100 2900 50  0001 C CNN
 	1    5100 2900
@@
 $EndComp
 $Comp
-L C C?
+L C C4
 U 1 1 5B22F803
 P 7450 3750
-F 0 "C?" H 7475 3850 50  0000 L CNN
+F 0 "C4" H 7475 3850 50  0000 L CNN
 F 1 "0.1uF" H 7475 3650 50  0000 L CNN
-F 2 "" H 7488 3600 50  0001 C CNN
+F 2 "Capacitors_SMD:C_0603_HandSoldering" H 7488 3600 50  0001 C CNN
 F 3 "" H 7450 3750 50  0001 C CNN
 	1    7450 3750
@@
 NoConn ~ 5950 6000
 $Comp
-L C C?
+L C C5
 U 1 1 5B22F9C7
 P 7850 2900
-F 0 "C?" H 7875 3000 50  0000 L CNN
+F 0 "C5" H 7875 3000 50  0000 L CNN
 F 1 "0.1uF" H 7875 2800 50  0000 L CNN
-F 2 "" H 7888 2750 50  0001 C CNN
+F 2 "Capacitors_SMD:C_0603_HandSoldering" H 7888 2750 50  0001 C CNN
 F 3 "" H 7850 2900 50  0001 C CNN
 	1    7850 2900
@@
 $EndComp
 $Comp
-L C C?
+L C C3
 U 1 1 5B22FCA2
 P 7450 2900
-F 0 "C?" H 7475 3000 50  0000 L CNN
+F 0 "C3" H 7475 3000 50  0000 L CNN
 F 1 "0.1uF" H 7475 2800 50  0000 L CNN
-F 2 "" H 7488 2750 50  0001 C CNN
+F 2 "Capacitors_SMD:C_0603_HandSoldering" H 7488 2750 50  0001 C CNN
 F 3 "" H 7450 2900 50  0001 C CNN
 	1    7450 2900
@@
 T1IN
 $Comp
-L VCC #PWR?
+L VCC #PWR02
 U 1 1 5B23086E
 P 8350 3800
-F 0 "#PWR?" H 8350 3650 50  0001 C CNN
+F 0 "#PWR02" H 8350 3650 50  0001 C CNN
 F 1 "VCC" H 8350 3950 50  0000 C CNN
 F 2 "" H 8350 3800 50  0001 C CNN
@@
 $EndComp
 $Comp
-L Conn_01x06_Male J?
+L Conn_01x06_Male J2
 U 1 1 5B230A0C
 P 8800 4300
-F 0 "J?" H 8800 4600 50  0000 C CNN
+F 0 "J2" H 8800 4600 50  0000 C CNN
 F 1 "USB" H 8800 3900 50  0000 C CNN
-F 2 "" H 8800 4300 50  0001 C CNN
+F 2 "Pin_Headers:Pin_Header_Straight_1x06_Pitch2.54mm" H 8800 4300 50  0001 C CNN
 F 3 "" H 8800 4300 50  0001 C CNN
 	1    8800 4300
@@
 $EndComp
 $Comp
-L GND #PWR?
+L GND #PWR03
 U 1 1 5B230BC2
 P 8450 4750
-F 0 "#PWR?" H 8450 4500 50  0001 C CNN
+F 0 "#PWR03" H 8450 4500 50  0001 C CNN
 F 1 "GND" H 8450 4600 50  0000 C CNN
 F 2 "" H 8450 4750 50  0001 C CNN
@@
 $EndComp
 $Comp
-L Jumper JP?
+L Jumper JP1
 U 1 1 5B230CB0
 P 8150 5100
-F 0 "JP?" H 8150 5250 50  0000 C CNN
+F 0 "JP1" H 8150 5250 50  0000 C CNN
 F 1 "Reset" H 8150 5020 50  0000 C CNN
-F 2 "" H 8150 5100 50  0001 C CNN
+F 2 "Pin_Headers:Pin_Header_Straight_1x02_Pitch2.54mm" H 8150 5100 50  0001 C CNN
 F 3 "" H 8150 5100 50  0001 C CNN
 	1    8150 5100
@@
 $EndComp
 $Comp
-L GND #PWR?
+L GND #PWR04
 U 1 1 5B230DB7
 P 8150 5550
-F 0 "#PWR?" H 8150 5300 50  0001 C CNN
+F 0 "#PWR04" H 8150 5300 50  0001 C CNN
 F 1 "GND" H 8150 5400 50  0000 C CNN
 F 2 "" H 8150 5550 50  0001 C CNN
@@
 $EndComp
 $Comp
-L MAX232 U?
+L MAX232 U1
 U 1 1 5B230F17
 P 6100 3650
-F 0 "U?" H 6000 4775 50  0000 R CNN
+F 0 "U1" H 6000 4775 50  0000 R CNN
 F 1 "MAX232" H 6000 4700 50  0000 R CNN
-F 2 "" H 6150 2600 50  0001 L CNN
+F 2 "Housings_SOIC:SOIC-16W_5.3x10.2mm_Pitch1.27mm" H 6150 2600 50  0001 L CNN
 F 3 "" H 6100 3750 50  0001 C CNN
 	1    6100 3650
@@
 $EndComp
 $Comp
-L GND #PWR?
+L GND #PWR05
 U 1 1 5B231623
 P 7450 4050
-F 0 "#PWR?" H 7450 3800 50  0001 C CNN
+F 0 "#PWR05" H 7450 3800 50  0001 C CNN
 F 1 "GND" H 7450 3900 50  0000 C CNN
 F 2 "" H 7450 4050 50  0001 C CNN
@@
 $EndComp
 $Comp
-L VCC #PWR?
+L VCC #PWR06
 U 1 1 5B2316E3
 P 6100 2250
-F 0 "#PWR?" H 6100 2100 50  0001 C CNN
+F 0 "#PWR06" H 6100 2100 50  0001 C CNN
 F 1 "VCC" H 6100 2400 50  0000 C CNN
 F 2 "" H 6100 2250 50  0001 C CNN
@@
 $EndComp
 $Comp
-L GND #PWR?
+L GND #PWR07
 U 1 1 5B231983
 P 7850 3150
-F 0 "#PWR?" H 7850 2900 50  0001 C CNN
+F 0 "#PWR07" H 7850 2900 50  0001 C CNN
 F 1 "GND" H 7850 3000 50  0000 C CNN
 F 2 "" H 7850 3150 50  0001 C CNN
@@
 $EndComp
 $Comp
-L VCC #PWR?
+L VCC #PWR08
 U 1 1 5B231F37
 P 7650 2250
-F 0 "#PWR?" H 7650 2100 50  0001 C CNN
+F 0 "#PWR08" H 7650 2100 50  0001 C CNN
 F 1 "VCC" H 7650 2400 50  0000 C CNN
 F 2 "" H 7650 2250 50  0001 C CNN
@@
 	4200 2900 4050 2900
 $Comp
-L GND #PWR?
+L GND #PWR09
 U 1 1 5B2328FB
 P 6100 5000
-F 0 "#PWR?" H 6100 4750 50  0001 C CNN
+F 0 "#PWR09" H 6100 4750 50  0001 C CNN
 F 1 "GND" H 6100 4850 50  0000 C CNN
 F 2 "" H 6100 5000 50  0001 C CNN
@@
 	1    0    0    -1
 $EndComp
+$Comp
+L PWR_FLAG #FLG010
+U 1 1 5B249AB0
+P 8000 2250
+F 0 "#FLG010" H 8000 2325 50  0001 C CNN
+F 1 "PWR_FLAG" H 8000 2400 50  0000 C CNN
+F 2 "" H 8000 2250 50  0001 C CNN
+F 3 "" H 8000 2250 50  0001 C CNN
+	1    8000 2250
+	1    0    0    -1
+$EndComp
+Wire Wire Line
+	8000 2250 8000 2350
+Wire Wire Line
+	8000 2350 7650 2350
+Connection ~ 7650 2350
+$Comp
+L PWR_FLAG #FLG011
+U 1 1 5B249BAC
+P 4800 3650
+F 0 "#FLG011" H 4800 3725 50  0001 C CNN
+F 1 "PWR_FLAG" H 4800 3800 50  0000 C CNN
+F 2 "" H 4800 3650 50  0001 C CNN
+F 3 "" H 4800 3650 50  0001 C CNN
+	1    4800 3650
+	1    0    0    -1
+$EndComp
+Wire Wire Line
+	4800 3650 4800 3800
+Wire Wire Line
+	4800 3800 4550 3800
+Connection ~ 4550 3800
 $EndSCHEMATC
